File: hardware/design/vis-analog-out/vis-analog-out.brd (EAGLE design)
At the start: 14 x 18 mm, 6 parts, among them J1 FH12-8S-0.5SH(55), U1 Chromation-optical-die-in-QFN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

Commit message: Consolidate EAGLE libraries into hardware/design/lbr
Parts:
- U1: value Chromation-optical-die-in-QFN-48-QuikPak-500580 -> CUVV-45-1-1-1-SMT
Changed lines of the file:
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@@
 <attribute name="VENDOR1_PQ_00001" value="1.54" x="8.6" y="14.8" size="1.778" layer="27" display="off"/>
 </element>
-<element name="U1" library="VIS-PKG" package="VIS-PKG" override_package3d_urn="urn:adsk.eagle:package:12144447/8" override_package_urn="urn:adsk.eagle:footprint:12144448/2" value="Chromation-optical-die-in-QFN-48-QuikPak-500580" x="10" y="5.91" smashed="yes" rot="MR0">
+<element name="U1" library="VIS-PKG" package="VIS-PKG" override_package3d_urn="urn:adsk.eagle:package:12144447/8" override_package_urn="urn:adsk.eagle:footprint:12144448/2" value="CUVV-45-1-1-1-SMT" x="10" y="5.91" smashed="yes" rot="MR0">
 <attribute name="EXPORT" value="YES" x="10" y="5.91" size="1.778" layer="28" rot="MR0" display="off"/>
 <attribute name="MANUF" value="Chromation" x="10" y="5.91" size="1.778" layer="28" rot="MR0" display="off"/>
-<attribute name="MANUF_PNUM" value="Spectrometer" x="10" y="5.91" size="1.778" layer="28" rot="MR0" display="off"/>
+<attribute name="MANUF_PNUM" value="CUVV-45-1-1-1-SMT" x="10" y="5.91" size="1.778" layer="28" rot="MR0" display="off"/>
 <attribute name="NAME" x="11.1" y="3.01" size="1.016" layer="28" font="vector" ratio="18" rot="MR0"/>
 <attribute name="NOTES" value="--" x="10" y="5.91" size="1.778" layer="28" rot="MR0" display="off"/>
 <attribute name="VALUE" x="15" y="5.91" size="1.016" layer="28" ratio="10" rot="MR0" align="center-right"/>
 <attribute name="VENDOR1" value="Chromation" x="10" y="5.91" size="1.778" layer="28" rot="MR0" display="off"/>
-<attribute name="VENDOR1_PNUM" value="Spectrometer" x="10" y="5.91" size="1.778" layer="28" rot="MR0" display="off"/>
+<attribute name="VENDOR1_PNUM" value="CUVV-45-1-1-1-SMT" x="10" y="5.91" size="1.778" layer="28" rot="MR0" display="off"/>
 <attribute name="VENDOR1_PQ_00001" value="--" x="10" y="5.91" size="1.778" layer="28" rot="MR0" display="off"/>
 </element>
